Commit message: TDM-30: root the sim URDF at base_link, base_footprint as its child
The EKF (state_estimation) publishes odom -> base_link, so the URDF's
base_footprint -> base_link gave base_link two TF parents and orphaned
base_footprint. Same fix as delivery-robo's robot_description (TDM-20):
base_joint is now base_link -> base_footprint at z = -wheel_radius
(-0.15); every other offset is unchanged, so base_footprint still sits
on the ground.

robot.urdf is regenerated from the xacro. robot.sdf is deliberately not:
Gazebo's link names never reach ROS TF, so the Gazebo model (root link,
spawn height, wheels, Ackermann plugin, ground truth) is untouched.
Regenerating it would re-root the model at base_link and raise
/ground_truth/odom z by 0.15 m; the xacro comment says so.

Checked on ROS_DOMAIN_ID=81 with robot_state_publisher + a fake 10 Hz
odom -> base_link at (1, 2, 0): odom -> base_footprint = (1, 2, -0.15),
base_footprint -> lidar_link = (0.3, 0, 0.3). The old URDF fails both
lookups (unconnected trees). In Gazebo this alone is not enough, see the
next commit.

Co-Authored-By: Claude Opus 5.5 <noreply@anthropic.com>
Claude-Session: https://claude.ai/code/session_019uGWZBNY4vkvV4wHR6a1at

File: src/simulation/urdf/robot.urdf (robot description, URDF)
Before this commit: robot delivery_robot, 12 links, 11 joints
Joints:
- joint base_joint: child base_link -> base_footprint; origin xyz=0 0 0.15 rpy=0 0 0 -> xyz=0 0 -0.15 rpy=0 0 0; parent base_footprint -> base_link

File: src/simulation/urdf/robot.urdf.xacro (robot description, xacro)
@@ -24,5 +24,4 @@
   </inertial>
 </xacro:macro>
-<link name="base_footprint"/>
 <link name="base_link">
   <visual>
@@ -39,8 +38,20 @@
   <xacro:box_inertia m="${chassis_mass}" w="${chassis_width}" h="${chassis_height}" d="${chassis_length}"/>
 </link>
+<!-- base_link is the root link, as in delivery-robo's robot_description: the
+     EKF (state_estimation) publishes odom -> base_link, so a base_footprint ->
+     base_link joint here would give base_link two TF parents and orphan
+     base_footprint. base_footprint hangs wheel_radius below base_link, on the
+     ground. robot_state_publisher warns that the root link has an inertia
+     (KDL ignores it); that is expected, don't add a dummy root to silence it.
+     robot.sdf was not regenerated for this and is still rooted at
+     base_footprint: Gazebo's link names never reach ROS TF. Regenerating it
+     re-roots the Gazebo model at base_link with the same geometry and inertia
+     (checked by diff, not run), so its model frame moves up 0.15 m to the
+     chassis centre and /ground_truth/odom z reads 0.15 m higher. -->
+<link name="base_footprint"/>
 <joint name="base_joint" type="fixed">
-  <parent link="base_footprint"/>
-  <child link="base_link"/>
-  <origin xyz="0 0 ${wheel_radius}" rpy="0 0 0"/>
+  <parent link="base_link"/>
+  <child link="base_footprint"/>
+  <origin xyz="0 0 ${-wheel_radius}" rpy="0 0 0"/>
 </joint>
 <xacro:macro name="rear_wheel" params="prefix y_offset">
